File: pcb/btmdpcb/power_mc34063.kicad_sch (KiCad schematic)
At the start: 13 parts, among them U6 MC34063AD

Commit message: Clean up schematic, implement all logic functionality
Parts:
- renumbered D2 to D1, L2 to L1, R18 to R14, R19 to R15, U6 to U1
Changed lines of the file:
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@@
 		(on_board yes)
 		(dnp no)
-		(property "Reference" "D2"
+		(property "Reference" "D1"
 			(at 167.64 89.8524 90)
 			(effects
@@
 			(project "btmdpcb"
 				(path "/6e43e92f-e106-411c-86ee-217d084aee5b/8d690d3f-f0ef-41aa-bdc4-e5b210b3f5fe"
-					(reference "D2")
+					(reference "D1")
 					(unit 1)
 				)
@@
 		(on_board yes)
 		(dnp no)
-		(property "Reference" "U6"
+		(property "Reference" "U1"
 			(at 137.16 68.58 0)
 			(effects
@@
 			(project "btmdpcb"
 				(path "/6e43e92f-e106-411c-86ee-217d084aee5b/8d690d3f-f0ef-41aa-bdc4-e5b210b3f5fe"
-					(reference "U6")
+					(reference "U1")
 					(unit 1)
 				)
@@
 		(dnp no)
 		(fields_autoplaced yes)
-		(property "Reference" "R19"
+		(property "Reference" "R15"
 			(at 182.88 91.4399 0)
 			(effects
@@
 			(project "btmdpcb"
 				(path "/6e43e92f-e106-411c-86ee-217d084aee5b/8d690d3f-f0ef-41aa-bdc4-e5b210b3f5fe"
-					(reference "R19")
+					(reference "R15")
 					(unit 1)
 				)
@@
 		(dnp no)
 		(fields_autoplaced yes)
-		(property "Reference" "R18"
+		(property "Reference" "R14"
 			(at 182.88 78.7399 0)
 			(effects
@@
 			(project "btmdpcb"
 				(path "/6e43e92f-e106-411c-86ee-217d084aee5b/8d690d3f-f0ef-41aa-bdc4-e5b210b3f5fe"
-					(reference "R18")
+					(reference "R14")
 					(unit 1)
 				)
@@
 		(on_board yes)
 		(dnp no)
-		(property "Reference" "L2"
+		(property "Reference" "L1"
 			(at 187.96 66.04 90)
 			(effects
@@
 			(project "btmdpcb"
 				(path "/6e43e92f-e106-411c-86ee-217d084aee5b/8d690d3f-f0ef-41aa-bdc4-e5b210b3f5fe"
-					(reference "L2")
-					(unit 1)
-				)
+					(reference "L1")
+					(unit 1)
+				)
