File: pcb/btmdpcb/power_we.kicad_sch (KiCad schematic)
At the start: 6 parts, among them U8 Würth 171010502

Commit message: Clean up schematic, implement all logic functionality
Parts:
- renumbered U8 to U3
Changed lines of the file:
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@@
 		(dnp no)
 		(fields_autoplaced yes)
-		(property "Reference" "U8"
+		(property "Reference" "U3"
 			(at 128.27 58.42 0)
 			(effects
@@
 			(project "btmdpcb"
 				(path "/6e43e92f-e106-411c-86ee-217d084aee5b/f98f56bc-3a06-4980-9f89-01c85da426aa"
-					(reference "U8")
+					(reference "U3")
 					(unit 1)
 				)

Commit message: Remove redundant regulators, simplify schematic
Parts:
- renumbered U3 to U1
Changed lines of the file:
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@@
 		(dnp no)
 		(fields_autoplaced yes)
-		(property "Reference" "U3"
+		(property "Reference" "U1"
 			(at 128.27 58.42 0)
 			(effects
@@
 			(project "btmdpcb"
 				(path "/6e43e92f-e106-411c-86ee-217d084aee5b/f98f56bc-3a06-4980-9f89-01c85da426aa"
-					(reference "U3")
+					(reference "U1")
 					(unit 1)
 				)
@@
 		(dnp no)
 		(fields_autoplaced yes)
-		(property "Reference" "#FLG03"
+		(property "Reference" "#FLG01"
 			(at 96.52 65.405 0)
 			(effects
@@
 			(project ""
 				(path "/6e43e92f-e106-411c-86ee-217d084aee5b/f98f56bc-3a06-4980-9f89-01c85da426aa"
-					(reference "#FLG03")
+					(reference "#FLG01")
 					(unit 1)
 				)

Commit message: Add BT auto-powerup (RC circuit + comparator)
Parts:
- renumbered R3fbt1 to R11, R3fbb1 to R12
Changed lines of the file:
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@@
 		(dnp no)
 		(fields_autoplaced yes)
-		(property "Reference" "R3fbt1"
+		(property "Reference" "R11"
 			(at 148.59 72.3899 0)
 			(effects
@@
 			(project "btmdpcb"
 				(path "/6e43e92f-e106-411c-86ee-217d084aee5b/f98f56bc-3a06-4980-9f89-01c85da426aa"
-					(reference "R3fbt1")
+					(reference "R11")
 					(unit 1)
 				)
@@
 		(dnp no)
 		(fields_autoplaced yes)
-		(property "Reference" "R3fbb1"
+		(property "Reference" "R12"
 			(at 148.59 88.8999 0)
 			(effects
@@
 			(project "btmdpcb"
 				(path "/6e43e92f-e106-411c-86ee-217d084aee5b/f98f56bc-3a06-4980-9f89-01c85da426aa"
-					(reference "R3fbb1")
+					(reference "R12")
 					(unit 1)
 				)

Commit message: Add missing libraries, assign all footprints
Parts:
- C3ff1: footprint Capacitor_SMD:C_0603_1608Metric_Pad1.08x0.95mm_HandSolder -> Capacitor_SMD:C_0402_1005Metric_Pad0.74x0.62mm_HandSolder
- renumbered R11 to R15, R12 to R16, U1 to U2
Changed lines of the file:
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@@
 		(dnp no)
 		(fields_autoplaced yes)
-		(property "Reference" "U1"
+		(property "Reference" "U2"
 			(at 128.27 58.42 0)
 			(effects
@@
 			(project "btmdpcb"
 				(path "/6e43e92f-e106-411c-86ee-217d084aee5b/f98f56bc-3a06-4980-9f89-01c85da426aa"
-					(reference "U1")
+					(reference "U2")
 					(unit 1)
 				)
@@
 			)
 		)
-		(property "Footprint" "Capacitor_SMD:C_0603_1608Metric_Pad1.08x0.95mm_HandSolder"
+		(property "Footprint" "Capacitor_SMD:C_0402_1005Metric_Pad0.74x0.62mm_HandSolder"
 			(at 160.9852 77.47 0)
 			(effects
@@
 		(dnp no)
 		(fields_autoplaced yes)
-		(property "Reference" "R11"
+		(property "Reference" "R15"
 			(at 148.59 72.3899 0)
 			(effects
@@
 			(project "btmdpcb"
 				(path "/6e43e92f-e106-411c-86ee-217d084aee5b/f98f56bc-3a06-4980-9f89-01c85da426aa"
-					(reference "R11")
+					(reference "R15")
 					(unit 1)
 				)
@@
 		(dnp no)
 		(fields_autoplaced yes)
-		(property "Reference" "R12"
+		(property "Reference" "R16"
 			(at 148.59 88.8999 0)
 			(effects
@@
 			(project "btmdpcb"
 				(path "/6e43e92f-e106-411c-86ee-217d084aee5b/f98f56bc-3a06-4980-9f89-01c85da426aa"
-					(reference "R12")
-					(unit 1)
-				)
+					(reference "R16")
+					(unit 1)
+				)

Commit message: Layout PCB
Parts:
- added C6: 1u, Capacitor_SMD:C_0805_2012Metric_Pad1.18x1.45mm_HandSolder, symbol Device:C
- added TP8: 1V5_IN, TestPoint:TestPoint_Pad_D1.0mm, symbol Connector:TestPoint
- added TP9: 1V5_OUT, TestPoint:TestPoint_Pad_D1.0mm, symbol Connector:TestPoint
- renumbered C3in1 to C5, C3ff1 to C7, C3out1 to C8, R15 to R21, R16 to R22, U2 to U3
Connections:
- net EN: now also C6.1
- net GND: now also C6.2
- net Vin: now also TP8.1
- net Vout: now also TP9.1
