File: pcb/btmdpcb/btmdpcb.kicad_sch (KiCad schematic)
At the start: 27 parts, among them Q1 BSD235N, Q2 BSD235C, Q3 BSD235N, Q4 BSD235C, U1 LM393

Commit message: Fix connectors & clearance; touch up PCB
Parts:
- added J1: AudioJack3_SwitchTR, symbol Connector_Audio:AudioJack3_SwitchTR
Connections:
- net MD unit (MZ-N505)/AUDIO_GND: now also J1.S
- net MD unit (MZ-N505)/AUDIO_L: now also J1.T
- net MD unit (MZ-N505)/AUDIO_R: now also J1.R
- no-connect marks 8 -> 10
Changed lines of the file:
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@@
+	)
+	(junction
+		(at 265.43 203.2)
+		(diameter 0)
+		(color 0 0 0 0)
 	)
 	(junction
@@
 	)
 	(junction
+		(at 257.81 195.58)
+		(diameter 0)
+		(color 0 0 0 0)
+	)
+	(junction
 		(at 340.36 50.8)
 		(diameter 0)
@@
 	)
 	(junction
+		(at 262.89 199.39)
+		(diameter 0)
+		(color 0 0 0 0)
+	)
+	(junction
 		(at 340.36 34.29)
 		(diameter 0)
@@
 		(diameter 0)
 		(color 0 0 0 0)
+	)
+	(no_connect
+		(at 260.35 190.5)
 	)
 	(no_connect
@@
 	)
 	(no_connect
+		(at 255.27 190.5)
+	)
+	(no_connect
 		(at 182.88 133.35)
 	)
@@
 	(wire
 		(pts
-			(xy 234.95 203.2) (xy 330.2 203.2)
+			(xy 234.95 203.2) (xy 265.43 203.2)
 		)
 		(stroke
@@
 	(wire
 		(pts
+			(xy 262.89 190.5) (xy 262.89 199.39)
+		)
+		(stroke
+			(width 0)
+			(type default)
+		)
+	)
+	(wire
+		(pts
 			(xy 354.33 102.87) (xy 354.33 105.41)
 		)
@@
 	(wire
 		(pts
+			(xy 265.43 190.5) (xy 265.43 203.2)
+		)
+		(stroke
+			(width 0)
+			(type default)
+		)
+	)
+	(wire
+		(pts
 			(xy 133.35 260.35) (xy 144.78 260.35)
 		)
@@
 	(wire
 		(pts
+			(xy 262.89 199.39) (xy 330.2 199.39)
+		)
+		(stroke
+			(width 0)
+			(type default)
+		)
+	)
+	(wire
+		(pts
 			(xy 289.56 86.36) (xy 289.56 148.59)
 		)
@@
 	(wire
 		(pts
-			(xy 234.95 195.58) (xy 330.2 195.58)
+			(xy 234.95 195.58) (xy 257.81 195.58)
 		)
 		(stroke
@@
 	(wire
 		(pts
+			(xy 257.81 190.5) (xy 257.81 195.58)
+		)
+		(stroke
+			(width 0)
+			(type default)
+		)
+	)
+	(wire
+		(pts
 			(xy 175.26 234.95) (xy 175.26 238.76)
 		)
@@
 	(wire
 		(pts
+			(xy 257.81 195.58) (xy 330.2 195.58)
+		)
+		(stroke
+			(width 0)
+			(type default)
+		)
+	)
+	(wire
+		(pts
 			(xy 133.35 46.99) (xy 133.35 38.1)
 		)
@@
 	(wire
 		(pts
-			(xy 234.95 199.39) (xy 330.2 199.39)
+			(xy 234.95 199.39) (xy 262.89 199.39)
 		)
 		(stroke
@@
 		(pts
 			(xy 146.05 29.21) (xy 154.94 29.21)
+		)
+		(stroke
+			(width 0)
+			(type default)
+		)
+	)
+	(wire
+		(pts
+			(xy 265.43 203.2) (xy 330.2 203.2)
 		)
 		(stroke
@@
 					(unit 1)
 				)
+			)
+		)
+	)
+	(symbol
+		(lib_id "Connector_Audio:AudioJack3_SwitchTR")
+		(at 262.89 185.42 270)
+		(unit 1)
+		(exclude_from_sim no)
+		(in_bom yes)
+		(on_board no)
+		(dnp yes)
+		(fields_autoplaced yes)
+		(property "Reference" "J1"
+			(at 267.97 182.2449 90)
+			(effects
+				(font
+					(size 1.27 1.27)
+				)
+				(justify left)
+			)
+		)
+		(property "Value" "AudioJack3_SwitchTR"
+			(at 267.97 184.7849 90)
+			(effects
+				(font
+					(size 1.27 1.27)
+				)
+				(justify left)
+			)
+		)
+		(property "Footprint" ""
+			(at 262.89 185.42 0)
+			(effects
+				(font
+					(size 1.27 1.27)
+				)
+				(hide yes)
+			)
+		)
+		(property "Datasheet" "~"
+			(at 262.89 185.42 0)
+			(effects
+				(font
+					(size 1.27 1.27)
+				)
+				(hide yes)
+			)
+		)
+		(property "Description" "Audio Jack, 3 Poles (Stereo / TRS), Switched TR Poles (Normalling)"
+			(at 262.89 185.42 0)
+			(effects
+				(font
+					(size 1.27 1.27)
+				)
+				(hide yes)
+			)
+		)
+		(pin "R"
+		)
+		(pin "TN"
+		)
+		(pin "T"
+		)
+		(pin "RN"
+		)
+		(pin "S"
+		)
+		(instances
+			(project ""
+				(path "/6e43e92f-e106-411c-86ee-217d084aee5b"
+					(reference "J1")
+					(unit 1)
+				)
